File: pcb_design/pcb_design.kicad_sch (KiCad schematic)
At the start: 5 parts, among them SW1 SW_Push, SW2 SW_Push, SW3 SW_Push, U1 MOUDLE-SEEEDUINO-XIAO, U2 ER_OLEDM0.91_1x-I2C

Commit message: Update PCB design files with layout adjustments and new STEP file
- Changed default plot path in `pcb_design.kicad_pro` to "./".
- Added new wire connections in `pcb_design.kicad_sch` for improved circuit layout.
- Reorganized existing wire connections and updated UUIDs for consistency.
- Adjusted symbol positions and properties for switches in `pcb_design.kicad_sch`.
- Introduced a new STEP file for 3D modeling of the PCB design.
Connections:
- net at SW3.1: now also U1.9 (PA7_A8_D8_SCK); no longer U1.11 (PA6_A10_D10_MOSI)
- net at SW1.1: now also U1.11 (PA6_A10_D10_MOSI); no longer U1.9 (PA7_A8_D8_SCK)
Other:
- moved on the sheet: SW1, SW3
Changed lines of the file:
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@@
+	(wire
+		(pts
+			(xy 166.37 129.54) (xy 172.72 129.54)
+		)
+		(stroke
+			(width 0)
+			(type default)
+		)
+	)
 	(wire
 		(pts
@@
 	(wire
 		(pts
-			(xy 166.37 129.54) (xy 172.72 129.54)
-		)
-		(stroke
-			(width 0)
-			(type default)
-		)
-	)
-	(wire
-		(pts
 			(xy 109.22 120.65) (xy 102.87 120.65)
 		)
@@
 	(wire
 		(pts
+			(xy 182.88 107.95) (xy 190.5 107.95)
+		)
+		(stroke
+			(width 0)
+			(type default)
+		)
+	)
+	(wire
+		(pts
 			(xy 102.87 120.65) (xy 102.87 85.09)
 		)
@@
 	(wire
 		(pts
+			(xy 182.88 129.54) (xy 190.5 129.54)
+		)
+		(stroke
+			(width 0)
+			(type default)
+		)
+	)
+	(wire
+		(pts
 			(xy 190.5 107.95) (xy 190.5 118.11)
 		)
@@
 	(wire
 		(pts
+			(xy 182.88 118.11) (xy 190.5 118.11)
+		)
+		(stroke
+			(width 0)
+			(type default)
+		)
+	)
+	(wire
+		(pts
+			(xy 156.21 110.49) (xy 152.4 110.49)
+		)
+		(stroke
+			(width 0)
+			(type default)
+		)
+	)
+	(wire
+		(pts
+			(xy 149.86 120.65) (xy 166.37 120.65)
+		)
+		(stroke
+			(width 0)
+			(type default)
+		)
+	)
+	(wire
+		(pts
+			(xy 109.22 118.11) (xy 105.41 118.11)
+		)
+		(stroke
+			(width 0)
+			(type default)
+		)
+	)
+	(wire
+		(pts
 			(xy 166.37 107.95) (xy 172.72 107.95)
-		)
-		(stroke
-			(width 0)
-			(type default)
-		)
-	)
-	(wire
-		(pts
-			(xy 182.88 107.95) (xy 190.5 107.95)
-		)
-		(stroke
-			(width 0)
-			(type default)
-		)
-	)
-	(wire
-		(pts
-			(xy 182.88 118.11) (xy 190.5 118.11)
-		)
-		(stroke
-			(width 0)
-			(type default)
-		)
-	)
-	(wire
-		(pts
-			(xy 156.21 110.49) (xy 152.4 110.49)
-		)
-		(stroke
-			(width 0)
-			(type default)
-		)
-	)
-	(wire
-		(pts
-			(xy 149.86 120.65) (xy 166.37 120.65)
-		)
-		(stroke
-			(width 0)
-			(type default)
-		)
-	)
-	(wire
-		(pts
-			(xy 109.22 118.11) (xy 105.41 118.11)
-		)
-		(stroke
-			(width 0)
-			(type default)
-		)
-	)
-	(wire
-		(pts
-			(xy 182.88 129.54) (xy 190.5 129.54)
 		)
 		(stroke
@@
 	(symbol
 		(lib_id "Switch:SW_Push")
-		(at 177.8 107.95 0)
+		(at 177.8 129.54 0)
 		(unit 1)
 		(body_style 1)
@@
 		(fields_autoplaced yes)
 		(property "Reference" "SW3"
-			(at 177.8 100.33 0)
+			(at 177.8 121.92 0)
 			(show_name no)
 			(do_not_autoplace no)
@@
 		)
 		(property "Value" "SW_Push"
-			(at 177.8 102.87 0)
+			(at 177.8 124.46 0)
 			(show_name no)
 			(do_not_autoplace no)
@@
 		)
 		(property "Footprint" "Button_Switch_Keyboard:SW_Cherry_MX_1.00u_PCB"
-			(at 177.8 102.87 0)
+			(at 177.8 124.46 0)
 			(hide yes)
 			(show_name no)
@@
 		)
 		(property "Datasheet" ""
-			(at 177.8 102.87 0)
+			(at 177.8 124.46 0)
 			(hide yes)
 			(show_name no)
@@
 		)
 		(property "Description" "Push button switch, generic, two pins"
-			(at 177.8 107.95 0)
+			(at 177.8 129.54 0)
 			(hide yes)
 			(show_name no)
@@
 	(symbol
 		(lib_id "Switch:SW_Push")
-		(at 177.8 129.54 0)
+		(at 177.8 107.95 0)
 		(unit 1)
 		(body_style 1)
@@
 		(fields_autoplaced yes)
 		(property "Reference" "SW1"
-			(at 177.8 121.92 0)
+			(at 177.8 100.33 0)
 			(show_name no)
 			(do_not_autoplace no)
@@
 		)
 		(property "Value" "SW_Push"
-			(at 177.8 124.46 0)
+			(at 177.8 102.87 0)
 			(show_name no)
 			(do_not_autoplace no)
@@
 		)
 		(property "Footprint" "Button_Switch_Keyboard:SW_Cherry_MX_1.00u_PCB"
-			(at 177.8 124.46 0)
+			(at 177.8 102.87 0)
 			(hide yes)
 			(show_name no)
@@
 		)
 		(property "Datasheet" ""
-			(at 177.8 124.46 0)
+			(at 177.8 102.87 0)
 			(hide yes)
 			(show_name no)
@@
 		)
 		(property "Description" "Push button switch, generic, two pins"
-			(at 177.8 129.54 0)
-			(hide yes)
-			(show_name no)
+			(at 177.8 107.95 0)
+			(hide yes)
+			(show_name no)
